Commit message: ur3e schmalz model updates

File: isaac_manipulator_pick_and_place/srdf/schmalz.srdf.xacro (robot description, xacro)
@@ -11,7 +11,4 @@
       <!--CHAINS - When a chain is specified, all the links along the chain (including endpoints) are included in the group. Additionally, all the joints that are parents to included links are also included. This means that joints along the chain and the parent joint of the base link are included in the group-->
       <!--SUBGROUPS - Groups can also be formed by referencing to already defined group names-->
-    <group name="schmalz_gripper">
-      <joint name="schmalz_base_link"/>
-    </group>
     <!--DISABLE COLLISIONS: By default it is assumed that any link of the robot could potentially come into collision with any other link in the robot. This tag disables collision checking between a specified pair of links. -->
     <disable_collisions link1="schmalz_base_link" link2="gripper_frame" reason="Never"/>
